File: kicad/mixeramp/mixeramp.kicad_pcb (KiCad board)
At the start: 2 copper layers, 44 parts, among them J1 Barrel_Jack_Switch, J2 AudioJack3, J3 AudioJack3, J4 AudioJack3, U2 L7809, U3 NJM4580

Commit message: add pcb
Parts:
- moved H4 129.5 mm to (164.3, 19.9)
- moved H2 101.6 mm to (164.3, 84.9)
- moved H3 81.0 mm to (99.3, 19.9)
- moved C10 58.8 mm to (126.6, 85.5), turned to 90 degrees
- moved H1 37.6 mm to (99.3, 84.9)
- moved R14 18.8 mm to (122.9, 41.5), turned to 180 degrees
- moved C13 17.0 mm to (126.0, 61.7)
- moved R6 10.7 mm to (133.9, 68.7)
- moved R2 10.7 mm to (126.9, 41.4)
- moved C14 9.25 mm to (126.1, 73.0)
- moved C6 9.16 mm to (148.0, 37.5)
- moved R5 7.69 mm to (153.5, 61.6)
- moved R3 7.69 mm to (148.5, 28.2)
- moved C11 7.69 mm to (155.4, 54.6)
- moved C12 7.69 mm to (155.4, 40.5)
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Routing:
- net GND: track 0.00 -> 293.1 mm, vias 0 -> 79
- net VCC: track 0.00 -> 177.4 mm
- net CH1_L: track 0.00 -> 47.8 mm
- net CH2_L: track 0.00 -> 40.1 mm
- net Net-(U3B--): track 0.00 -> 37.3 mm
- net CH1_R: track 0.00 -> 24.8 mm
- net OUT_L: track 0.00 -> 24.7 mm
- net Net-(C1-Pad2): track 0.00 -> 24.3 mm
- net Net-(U2-IN): track 0.00 -> 23.3 mm
- net CH2_R: track 0.00 -> 21.1 mm
- net Net-(U3B-+): track 0.00 -> 19.4 mm
- net Net-(U3A-+): track 0.00 -> 17.7 mm
- net OUT_R: track 0.00 -> 17.3 mm
- net Net-(C17-Pad2): track 0.00 -> 12.7 mm
- net Net-(U3A--): track 0.00 -> 12.5 mm
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- added copper zone on B.Cu, net GND
- added copper zone on F.Cu, net GND
Other:
- board outline added: 74 x 74 mm
